Commit message: blackbot is getting accurate calibrations!

File: blackbot_description/urdf/only_camera_system.urdf.xacro (robot description, xacro)
@@ -1,9 +1,9 @@
 <?xml version="1.0"?>
 <robot xmlns:xacro="http://www.ros.org/wiki/xacro" name="only_camera_system">
-<!--<link name="ptu_mount_link" />-->
+  <!--<link name="ptu_mount_link" />-->
   <!--Include a descritpion of the asus camera (from the hector_sensors_description package)-->
   <xacro:include filename="$(find blackbot_description)/urdf/kinect2.urdf.xacro"/>
   <!--Create the_camera instance, giving as input arguments the values for the estimated transformation-->
-  <xacro:kinect2_xacro prefix="camera" parent="ptu_mount_link">
+  <xacro:kinect2_xacro prefix="kinect2" parent="ptu_mount_link">
     <origin rpy="0 0 0" xyz="0 0 0"/>
   </xacro:kinect2_xacro>
