Commit message: changing default camera name from kinect2 to camera

File: blackbot_calibration/calibration/hand_in_eye.urdf.xacro (robot description, xacro)
@@ -2,11 +2,11 @@
 <robot xmlns:xacro="http://www.ros.org/wiki/xacro">
 <!--This xacro contains six xacro propperties representing a transformation obtained through calibration-->
-<!--Calibration generated at 15:34:25, 30/06/2016 -->
+<!--Calibration generated at 16:32:25, 30/06/2016 -->
 <!--This file was written automatically using the "rosrun blackbot_calibration store_calibration" command. -->
-<xacro:property name="roll" value="-1.31851218837"/>
-<xacro:property name="pitch" value="0.00399881683654"/>
-<xacro:property name="yaw" value="-1.54629208765"/>
-<xacro:property name="x" value="0.0164651946802"/>
-<xacro:property name="y" value="-0.0812336964619"/>
-<xacro:property name="z" value="0.0329665095287"/>
+<xacro:property name="roll" value="-1.3190537844"/>
+<xacro:property name="pitch" value="0.00340101049727"/>
+<xacro:property name="yaw" value="-1.53479744513"/>
+<xacro:property name="x" value="0.0163624272899"/>
+<xacro:property name="y" value="-0.0802404630618"/>
+<xacro:property name="z" value="0.0340890188704"/>
 </robot>

File: blackbot_description/urdf/calibrated_system.urdf.xacro (robot description, xacro)
@@ -13,5 +13,5 @@
   <xacro:ptu_d46 name="ptu"/>
   <!--Create the_camera instance, giving as input arguments the values for the estimated transformation-->
-  <xacro:kinect2_xacro prefix="kinect2" parent="ptu_mount_link">
+  <xacro:kinect2_xacro prefix="camera" parent="ptu_mount_link">
     <origin rpy="0 0 0" xyz="0 0 0"/>
   </xacro:kinect2_xacro>
@@ -22,5 +22,5 @@
     <origin rpy="${roll} ${pitch} ${yaw}" xyz="${x} ${y} ${z}"/>
     <parent link="ptu_mount_link"/>
-    <child link="kinect2_rgb_optical_frame"/>
+    <child link="camera_rgb_optical_frame"/>
   </joint>
 </robot>

File: blackbot_description/urdf/only_camera_system.urdf.xacro (robot description, xacro)
@@ -5,5 +5,5 @@
   <xacro:include filename="$(find blackbot_description)/urdf/kinect2.urdf.xacro"/>
   <!--Create the_camera instance, giving as input arguments the values for the estimated transformation-->
-  <xacro:kinect2_xacro prefix="kinect2" parent="ptu_mount_link">
+  <xacro:kinect2_xacro prefix="camera" parent="ptu_mount_link">
     <origin rpy="0 0 0" xyz="0 0 0"/>
   </xacro:kinect2_xacro>

Commit message: new hand in eye calibration

File: blackbot_calibration/calibration/hand_in_eye.urdf.xacro (robot description, xacro)
@@ -2,11 +2,11 @@
 <robot xmlns:xacro="http://www.ros.org/wiki/xacro">
 <!--This xacro contains six xacro propperties representing a transformation obtained through calibration-->
-<!--Calibration generated at 16:32:25, 30/06/2016 -->
+<!--Calibration generated at 14:59:44, 18/07/2016 -->
 <!--This file was written automatically using the "rosrun blackbot_calibration store_calibration" command. -->
-<xacro:property name="roll" value="-1.3190537844"/>
-<xacro:property name="pitch" value="0.00340101049727"/>
-<xacro:property name="yaw" value="-1.53479744513"/>
-<xacro:property name="x" value="0.0163624272899"/>
-<xacro:property name="y" value="-0.0802404630618"/>
-<xacro:property name="z" value="0.0340890188704"/>
+<xacro:property name="roll" value="-1.32523001314"/>
+<xacro:property name="pitch" value="0.00264550898646"/>
+<xacro:property name="yaw" value="-1.54662677263"/>
+<xacro:property name="x" value="0.019628550271"/>
+<xacro:property name="y" value="-0.0915189463546"/>
+<xacro:property name="z" value="0.0455779558533"/>
 </robot>

Commit message: new hand in eye calibration

File: blackbot_calibration/calibration/hand_in_eye.urdf.xacro (robot description, xacro)
@@ -2,11 +2,11 @@
 <robot xmlns:xacro="http://www.ros.org/wiki/xacro">
 <!--This xacro contains six xacro propperties representing a transformation obtained through calibration-->
-<!--Calibration generated at 14:59:44, 18/07/2016 -->
+<!--Calibration generated at 15:32:24, 05/09/2016 -->
 <!--This file was written automatically using the "rosrun blackbot_calibration store_calibration" command. -->
-<xacro:property name="roll" value="-1.32523001314"/>
-<xacro:property name="pitch" value="0.00264550898646"/>
-<xacro:property name="yaw" value="-1.54662677263"/>
-<xacro:property name="x" value="0.019628550271"/>
-<xacro:property name="y" value="-0.0915189463546"/>
-<xacro:property name="z" value="0.0455779558533"/>
+<xacro:property name="roll" value="-1.3211598456"/>
+<xacro:property name="pitch" value="0.00630137139324"/>
+<xacro:property name="yaw" value="-1.54555762024"/>
+<xacro:property name="x" value="0.019609299187"/>
+<xacro:property name="y" value="-0.0935113512419"/>
+<xacro:property name="z" value="0.0434518685604"/>
 </robot>

Commit message: new blackbot iai kinect2 and hand in eye calibration

File: blackbot_calibration/calibration/hand_in_eye.urdf.xacro (robot description, xacro)
@@ -2,11 +2,11 @@
 <robot xmlns:xacro="http://www.ros.org/wiki/xacro">
 <!--This xacro contains six xacro propperties representing a transformation obtained through calibration-->
-<!--Calibration generated at 15:32:24, 05/09/2016 -->
+<!--Calibration generated at 20:43:01, 17/11/2016 -->
 <!--This file was written automatically using the "rosrun blackbot_calibration store_calibration" command. -->
-<xacro:property name="roll" value="-1.3211598456"/>
-<xacro:property name="pitch" value="0.00630137139324"/>
-<xacro:property name="yaw" value="-1.54555762024"/>
-<xacro:property name="x" value="0.019609299187"/>
-<xacro:property name="y" value="-0.0935113512419"/>
-<xacro:property name="z" value="0.0434518685604"/>
+<xacro:property name="roll" value="-1.32733121928"/>
+<xacro:property name="pitch" value="0.0052155822955"/>
+<xacro:property name="yaw" value="-1.53585211679"/>
+<xacro:property name="x" value="0.0198154118647"/>
+<xacro:property name="y" value="-0.0935828470128"/>
+<xacro:property name="z" value="0.0467029473312"/>
 </robot>

Commit message: new calibration failed. Using the old one

File: blackbot_calibration/calibration/hand_in_eye.urdf.xacro (robot description, xacro)
@@ -2,11 +2,11 @@
 <robot xmlns:xacro="http://www.ros.org/wiki/xacro">
 <!--This xacro contains six xacro propperties representing a transformation obtained through calibration-->
-<!--Calibration generated at 20:43:01, 17/11/2016 -->
+<!--Calibration generated at 18:40:05, 25/11/2016 -->
 <!--This file was written automatically using the "rosrun blackbot_calibration store_calibration" command. -->
-<xacro:property name="roll" value="-1.32733121928"/>
-<xacro:property name="pitch" value="0.0052155822955"/>
-<xacro:property name="yaw" value="-1.53585211679"/>
-<xacro:property name="x" value="0.0198154118647"/>
-<xacro:property name="y" value="-0.0935828470128"/>
-<xacro:property name="z" value="0.0467029473312"/>
+<xacro:property name="roll" value="-1.32072575053"/>
+<xacro:property name="pitch" value="0.00825181300146"/>
+<xacro:property name="yaw" value="-1.53986148754"/>
+<xacro:property name="x" value="0.0196963760223"/>
+<xacro:property name="y" value="-0.0939720737455"/>
+<xacro:property name="z" value="0.0475767111504"/>
 </robot>

Commit message: new hand in eye calibration

File: blackbot_calibration/calibration/hand_in_eye.urdf.xacro (robot description, xacro)
@@ -2,11 +2,11 @@
 <robot xmlns:xacro="http://www.ros.org/wiki/xacro">
 <!--This xacro contains six xacro propperties representing a transformation obtained through calibration-->
-<!--Calibration generated at 18:40:05, 25/11/2016 -->
+<!--Calibration generated at 14:13:15, 27/12/2016 -->
 <!--This file was written automatically using the "rosrun blackbot_calibration store_calibration" command. -->
-<xacro:property name="roll" value="-1.32072575053"/>
-<xacro:property name="pitch" value="0.00825181300146"/>
-<xacro:property name="yaw" value="-1.53986148754"/>
-<xacro:property name="x" value="0.0196963760223"/>
-<xacro:property name="y" value="-0.0939720737455"/>
-<xacro:property name="z" value="0.0475767111504"/>
+<xacro:property name="roll" value="-1.32849754702"/>
+<xacro:property name="pitch" value="0.0241945633189"/>
+<xacro:property name="yaw" value="-1.54479678214"/>
+<xacro:property name="x" value="0.0261341559846"/>
+<xacro:property name="y" value="-0.0989153757223"/>
+<xacro:property name="z" value="0.0366027152118"/>
 </robot>

Commit message: latest calibration

File: blackbot_calibration/calibration/hand_in_eye.urdf.xacro (robot description, xacro)
@@ -2,11 +2,11 @@
 <robot xmlns:xacro="http://www.ros.org/wiki/xacro">
 <!--This xacro contains six xacro propperties representing a transformation obtained through calibration-->
-<!--Calibration generated at 14:13:15, 27/12/2016 -->
+<!--Calibration generated at 22:45:41, 10/05/2017 -->
 <!--This file was written automatically using the "rosrun blackbot_calibration store_calibration" command. -->
-<xacro:property name="roll" value="-1.32849754702"/>
-<xacro:property name="pitch" value="0.0241945633189"/>
-<xacro:property name="yaw" value="-1.54479678214"/>
-<xacro:property name="x" value="0.0261341559846"/>
-<xacro:property name="y" value="-0.0989153757223"/>
-<xacro:property name="z" value="0.0366027152118"/>
+<xacro:property name="roll" value="-0.00796440881548"/>
+<xacro:property name="pitch" value="-0.151422939784"/>
+<xacro:property name="yaw" value="-0.0222183295858"/>
+<xacro:property name="x" value="-0.0114470226192"/>
+<xacro:property name="y" value="0.0141832849622"/>
+<xacro:property name="z" value="0.107186444319"/>
 </robot>

File: blackbot_description/urdf/calibrated_system.urdf.xacro (robot description, xacro)
@@ -9,18 +9,18 @@
   <xacro:include filename="$(find blackbot_description)/urdf/d46.urdf.xacro"/>
   <!--Include a descritpion of the asus camera (from the hector_sensors_description package)-->
-  <xacro:include filename="$(find blackbot_description)/urdf/kinect2.urdf.xacro"/>
+  <!--<xacro:include filename="$(find blackbot_description)/urdf/kinect2.urdf.xacro"/>-->
   <!--Create a rnr_pan_tilt instance -->
   <xacro:ptu_d46 name="ptu"/>
   <!--Create the_camera instance, giving as input arguments the values for the estimated transformation-->
-  <xacro:kinect2_xacro prefix="camera" parent="ptu_mount_link">
-    <origin rpy="0 0 0" xyz="0 0 0"/>
-  </xacro:kinect2_xacro>
-  <joint name="camera_joint" type="fixed">
-    <!--This is given by the eye in hand calibration (Used up to December 17, 2015)-->
-    <!--<origin rpy="-0.014926 0.081221 0.002227" xyz="0.013207 0.007074 0.086040"/>-->
-    <!--<origin rpy="$(arg roll) $(arg pitch) $(arg yaw)" xyz="$(arg x) $(arg y) $(arg z)"/>-->
-    <origin rpy="${roll} ${pitch} ${yaw}" xyz="${x} ${y} ${z}"/>
-    <parent link="ptu_mount_link"/>
-    <child link="camera_rgb_optical_frame"/>
-  </joint>
+  <!--<xacro:kinect2_xacro prefix="camera" parent="ptu_mount_link">-->
+    <!--<origin rpy="0 0 0" xyz="0 0 0"/>-->
+  <!--</xacro:kinect2_xacro>-->
+  <!--<joint name="camera_joint" type="fixed">-->
+    <!--[>This is given by the eye in hand calibration (Used up to December 17, 2015)<]-->
+    <!--[><origin rpy="-0.014926 0.081221 0.002227" xyz="0.013207 0.007074 0.086040"/><]-->
+    <!--[><origin rpy="$(arg roll) $(arg pitch) $(arg yaw)" xyz="$(arg x) $(arg y) $(arg z)"/><]-->
+    <!--<origin rpy="${roll} ${pitch} ${yaw}" xyz="${x} ${y} ${z}"/>-->
+    <!--<parent link="ptu_mount_link"/>-->
+    <!--<child link="camera_rgb_optical_frame"/>-->
+  <!--</joint>-->
 </robot>
